File: hardware/macropad/macropad.kicad_pcb (KiCad board)
At the start: 2 copper layers, 126 x 99.5 mm, 7 parts, among them Q1 SW_Push

Commit message: Add Rotary Encoder
Parts:
- added REF**: MountingHole_3.2mm_M3, MountingHole:MountingHole_3.2mm_M3, F.Cu at (138.8, 120.7)
- added REF**: MountingHole_3.2mm_M3, MountingHole:MountingHole_3.2mm_M3, F.Cu at (46.9, 121.0)
- added REF**: MountingHole_3.2mm_M3, MountingHole:MountingHole_3.2mm_M3, F.Cu at (46.6, 32.6)
- added REF**: MountingHole_3.2mm_M3, MountingHole:MountingHole_3.2mm_M3, F.Cu at (138.9, 32.1)
- added volume_control1: RotaryEncoder_Switch, Rotary_Encoder:RotaryEncoder_Alps_EC11E-Switch_Vertical_H20mm, F.Cu at (114.0, 40.6)
- D1, E1, F1, Q1, R1, W1: moved to B.Cu
- moved F1 26.6 mm to (124.9, 101.5), turned to 180 degrees
- moved R1 25.3 mm to (114.3, 82.5), turned to 180 degrees
- moved D1 18.7 mm to (105.8, 101.5), turned to 180 degrees
- moved E1 17.7 mm to (95.2, 82.5), turned to 180 degrees
- moved W1 9.49 mm to (76.2, 82.5), turned to 180 degrees
- moved A1 6.02 mm to (66.5, 51.0)
- moved Q1 1.62 mm to (57.1, 82.5), turned to 180 degrees
Connections:
- A1 pad 12: unconnected-(A1-GPIO9-Pad12) -> Net-(A1-GPIO9)
- A1 pad 16: Net-(A1-GPIO12) -> unconnected-(A1-GPIO12-Pad16)
- A1 pad 22: Net-(A1-GPIO17) -> unconnected-(A1-GPIO17-Pad22)
- A1 pad 24: unconnected-(A1-GPIO18-Pad24)_1 -> Net-(A1-GPIO18)
- A1 pad 26: unconnected-(A1-GPIO20-Pad26) -> Net-(A1-GPIO20)
- A1 pad 7: unconnected-(A1-GPIO5-Pad7)_1 -> unconnected-(A1-GPIO5-Pad7)
- D1 pad 1: Net-(A1-GPIO12) -> Net-(A1-GPIO14)
- E1 pad 1: Net-(A1-GPIO13) -> Net-(A1-GPIO9)
- F1 pad 1: Net-(A1-GPIO16) -> Net-(A1-GPIO15)
- Q1 pad 1: Net-(A1-GPIO15) -> unconnected-(A1-GPIO1-Pad2)
- R1 pad 1: Net-(A1-GPIO17) -> Net-(A1-GPIO13)
- W1 pad 1: Net-(A1-GPIO14) -> unconnected-(A1-GPIO5-Pad7)
Routing:
- added copper zone on B.Cu, net GND
Other:
- board size 126 x 99.5 mm -> 103.6 x 99.8 mm

Commit message: Complete Back Copper Routing
Parts:
- removed the REF** at (138.8, 120.7)
- removed the REF** at (46.9, 121.0)
- removed the REF** at (138.9, 32.1)
- added REF**: MountingHole_3.2mm_M3, MountingHole:MountingHole_3.2mm_M3, F.Cu at (75.5, 163.8)
- added REF**: MountingHole_3.2mm_M3, MountingHole:MountingHole_3.2mm_M3, F.Cu at (163.8, 74.9)
- added REF**: MountingHole_3.2mm_M3, MountingHole:MountingHole_3.2mm_M3, F.Cu at (163.8, 163.8)
- moved D1 52.1 mm to (134.7, 144.9)
- moved F1 52.1 mm to (153.7, 144.9)
- moved volume_control1 52.1 mm to (142.9, 84.0)
- moved Q1 52.1 mm to (86.0, 125.8)
- moved REF** 52.1 mm to (75.5, 76.0)
- moved A1 52.1 mm to (95.3, 94.3)
- moved E1 52.1 mm to (124.1, 125.8)
- moved R1 52.1 mm to (143.2, 125.8)
- moved W1 52.1 mm to (105.0, 125.8)
Connections:
- A1 pad 21: Net-(A1-GPIO16) -> unconnected-(A1-GPIO16-Pad21)_1
- A1 pad 22: unconnected-(A1-GPIO17-Pad22) -> Net-(A1-GPIO17)
- A1 pad 24: Net-(A1-GPIO18) -> unconnected-(A1-GPIO18-Pad24)_1
- A1 pad 25: unconnected-(A1-GPIO19-Pad25) -> Net-(A1-GPIO19)
- D1 pad 1: Net-(A1-GPIO14) -> Net-(A1-GPIO13)
- F1 pad 1: Net-(A1-GPIO15) -> Net-(A1-GPIO14)
- R1 pad 1: Net-(A1-GPIO13) -> Net-(A1-GPIO15)
- volume_control1 pad A: Net-(A1-GPIO18) -> Net-(A1-GPIO19)
- volume_control1 pad B: Net-(A1-GPIO16) -> Net-(A1-GPIO17)
Routing:
- net GND: track 0.36 -> 73.4 mm
- net Net-(A1-GPIO20): track 0.00 -> 65.9 mm
- net Net-(A1-GPIO14): track 0.00 -> 51.4 mm
- net Net-(A1-GPIO13): track 0.00 -> 45.6 mm
- net Net-(A1-GPIO19): track 0.00 -> 39.6 mm
- net Net-(A1-GPIO17): track 0.00 -> 29.8 mm
- net Net-(A1-GPIO9): track 0.00 -> 27.5 mm
- net Net-(A1-GPIO15): track 0.00 -> 27.0 mm
- net unconnected-(A1-GPIO5-Pad7): track 0.00 -> 24.8 mm
- net unconnected-(A1-GPIO1-Pad2): track 0.00 -> 22.2 mm
Other:
- board size 103.6 x 99.8 mm -> 100 x 100 mm

Commit message: Pass Electrical & Design Rule Checks
Parts:
- moved REF** 1.02 mm to (75.5, 74.9)
Routing:
- net GND: track 73.4 -> 164.1 mm
Other:
- board text added: "A1"
Changed lines of the file:
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@@
 			(unlocked yes)
 			(layer "F.SilkS")
+			(hide yes)
 			(effects
 				(font
@@
 			)
 		)
-		(fp_text user "${REFERENCE}"
-			(at 0.2659 -1.13 0)
-			(layer "F.Fab")
-			(effects
-				(font
-					(size 1 1)
-					(thickness 0.15)
-				)
-			)
-		)
 		(pad "" np_thru_hole circle
 			(at -2.725 -24 90)
@@
 			(members "006d2d41-2d37-4c3b-8ade-2e374407b7d6" "17da24c6-d3f6-4235-afb7-ba9865c96812"
 				"1e71ca56-73f0-46e0-ac01-c9fed4d113d3" "22ad3a94-ae21-46a1-a9c3-3106f74e4a88"
-				"3b423084-40e8-42bb-b24f-7ce5831234a7" "3ced2804-9639-4fb3-9f91-04446302b402"
-				"49c6f62b-7dd3-4e9d-b733-d9ceebdff86c" "5514c5be-a6a1-40cf-9e63-db6d7c8b6bf4"
-				"5aa54d31-cb15-4e2a-b7cd-bb726a3fa818" "72e2a461-ed60-415a-8053-60b164c24008"
-				"8d1c3e33-c6a3-409d-a31c-08f2623c5676" "a3738ca6-3067-4bf4-ad66-12636c46534f"
-				"b596fe6e-ef53-439b-9137-8ed8270756d8" "bce3bde7-dc8f-4361-b63d-8f243d2a416d"
-				"bd813e4f-9c41-4cbc-a5c5-f5a999f68615" "c83808b3-66ab-4540-86b8-4ba7ca91e4cb"
-				"db566a3f-c356-413e-8329-eeda035a7f55" "dc0f3a58-d23b-47ed-8c02-3b4ab1f2ef69"
-				"dd1c4bf5-3388-4bc2-b31a-3e82d76fe683" "e0fa98a2-3544-4b22-b612-8d7d5dfef85b"
-				"e20a3d37-e2b8-498c-9931-22a8e0358bfe" "f448a00e-8e44-44ca-b319-246119b2d7b4"
+				"3b423084-40e8-42bb-b24f-7ce5831234a7" "49c6f62b-7dd3-4e9d-b733-d9ceebdff86c"
+				"5514c5be-a6a1-40cf-9e63-db6d7c8b6bf4" "5aa54d31-cb15-4e2a-b7cd-bb726a3fa818"
+				"72e2a461-ed60-415a-8053-60b164c24008" "8d1c3e33-c6a3-409d-a31c-08f2623c5676"
+				"a3738ca6-3067-4bf4-ad66-12636c46534f" "b596fe6e-ef53-439b-9137-8ed8270756d8"
+				"bce3bde7-dc8f-4361-b63d-8f243d2a416d" "bd813e4f-9c41-4cbc-a5c5-f5a999f68615"
+				"c83808b3-66ab-4540-86b8-4ba7ca91e4cb" "db566a3f-c356-413e-8329-eeda035a7f55"
+				"dc0f3a58-d23b-47ed-8c02-3b4ab1f2ef69" "dd1c4bf5-3388-4bc2-b31a-3e82d76fe683"
+				"e0fa98a2-3544-4b22-b612-8d7d5dfef85b" "e20a3d37-e2b8-498c-9931-22a8e0358bfe"
+				"f448a00e-8e44-44ca-b319-246119b2d7b4"
 			)
 		)
@@
 	(footprint "MountingHole:MountingHole_3.2mm_M3"
 		(layer "F.Cu")
-		(at 75.45 75.95)
+		(at 75.45 74.93)
 		(descr "Mounting Hole 3.2mm, M3, no annular, generated by kicad-footprint-generator mountinghole.py")
 		(tags "mountinghole M3")
@@
 	)
 	(gr_rect
-		(start 69.85 69.85)
-		(end 169.85 169.85)
+		(start 69.49 69.69)
+		(end 169.49 169.69)
 		(stroke
 			(width 0.05)
@@
 		(layer "Edge.Cuts")
 	)
+	(gr_text "A1"
+		(at 84.8125 94.35 0)
+		(layer "F.SilkS")
+		(effects
+			(font
+				(size 1 1)
+				(thickness 0.15)
+			)
+		)
+	)
 	(segment
 		(start 78.915 123.31)
@@
 	)
 	(segment
-		(start 93.467 120.77)
-		(end 93.467 120.407)
+		(start 91.842 120.77)
+		(end 91.842 118.782)
 		(width 0.2)
 		(layer "B.Cu")
@@
 	)
 	(segment
-		(start 91.842 120.77)
-		(end 91.842 118.782)
+		(start 157.4 84)
+		(end 154.9 86.5)
 		(width 0.2)
 		(layer "B.Cu")
@@
 	)
 	(segment
-		(start 157.4 84)
-		(end 154.9 86.5)
+		(start 113.3 86.56)
+		(end 114.4 85.46)
+		(width 0.2)
+		(layer "B.Cu")
+		(net "GND")
+	)
+	(segment
+		(start 101.7 86.46)
+		(end 102.87 87.63)
 		(width 0.2)
 		(layer "B.Cu")
@@
 	)
 	(segment
+		(start 90.1 102.14)
+		(end 100.6 102.14)
+		(width 0.2)
+		(layer "B.Cu")
+		(net "GND")
+	)
+	(segment
 		(start 119.85 80.01)
 		(end 136.41 80.01)
@@
 	)
 	(segment
+		(start 100.6 102.14)
+		(end 101.7 103.24)
+		(width 0.2)
+		(layer "B.Cu")
+		(net "GND")
+	)
+	(segment
+		(start 89 103.24)
+		(end 87.9 102.14)
+		(width 0.2)
+		(layer "B.Cu")
+		(net "GND")
+	)
+	(segment
 		(start 154.9 86.5)
 		(end 142.9 86.5)
@@
 	)
 	(segment
+		(start 102.8 86.56)
+		(end 113.3 86.56)
+		(width 0.2)
+		(layer "B.Cu")
+		(net "GND")
+	)
+	(segment
+		(start 113.3 102.14)
+		(end 114.4 103.24)
+		(width 0.2)
+		(layer "B.Cu")
+		(net "GND")
+	)
+	(segment
+		(start 101.7 85.46)
+		(end 102.8 86.56)
+		(width 0.2)
+		(layer "B.Cu")
+		(net "GND")
+	)
+	(segment
 		(start 136.41 80.01)
 		(end 142.9 86.5)
 		(width 0.2)
 		(layer "B.Cu")
+		(net "GND")
+	)
+	(segment
+		(start 102.87 102.07)
+		(end 101.7 103.24)
+		(width 0.2)
+		(layer "B.Cu")
+		(net "GND")
+	)
+	(segment
+		(start 102.87 102.07)
+		(end 102.8 102.14)
+		(width 0.2)
+		(layer "B.Cu")
+		(net "GND")
+	)
+	(segment
+		(start 77.4 102.14)
+		(end 76.3 103.24)
+		(width 0.2)
+		(layer "B.Cu")
+		(net "GND")
+	)
+	(segment
+		(start 89 103.24)
+		(end 90.1 102.14)
+		(width 0.2)
+		(layer "B.Cu")
+		(net "GND")
+	)
+	(segment
+		(start 87.9 102.14)
+		(end 77.4 102.14)
+		(width 0.2)
+		(layer "B.Cu")
+		(net "GND")
+	)
+	(segment
+		(start 102.8 102.14)
+		(end 113.3 102.14)
+		(width 0.2)
+		(layer "B.Cu")
+		(net "GND")
+	)
+	(segment
+		(start 101.7 103.24)
+		(end 102.8 102.14)
+		(width 0.2)
+		(layer "B.Cu")
+		(net "GND")
+	)
+	(segment
+		(start 101.7 85.46)
+		(end 101.7 86.46)
+		(width 0.2)
+		(layer "B.Cu")
+		(net "GND")
+	)
+	(segment
+		(start 76.3 85.46)
+		(end 76.3 103.24)
+		(width 0.2)
+		(layer "B.Cu")
+		(net "GND")
+	)
+	(segment
+		(start 102.87 87.63)
+		(end 102.87 102.07)
+		(width 0.2)
+		(layer "B.Cu")
