File: hardware/macropad/macropad.kicad_sch (KiCad schematic)
At the start: 0 parts

Commit message: KiCad PCB Layout
Parts:
- added A1: RaspberryPi_Pico, Module:RaspberryPi_Pico_Common_Unspecified, symbol MCU_Module:RaspberryPi_Pico
- added D1, E1, F1, Q1, R1, W1: SW_Push, MX_Hotswap:MX-Hotswap-1U, symbol Switch:SW_Push
Connections:
- new net: A1.22 (GPIO17), R1.1
- new net: A1.16 (GPIO12), D1.1
- new net: A1.20 (GPIO15), Q1.1
- new net: A1.17 (GPIO13), E1.1
- new net: A1.19 (GPIO14), W1.1
- new net: A1.21 (GPIO16), F1.1
- new net GND: A1.13 (GND), A1.18 (GND), A1.23 (GND), A1.28 (GND), A1.3 (GND), A1.38 (GND), A1.8 (GND), D1.2, E1.2, F1.2, Q1.2, R1.2, W1.2
- no-connect marks 0 -> 21

Commit message: Add Rotary Encoder
Parts:
- added volume_control1: RotaryEncoder_Switch, Rotary_Encoder:RotaryEncoder_Alps_EC11E-Switch_Vertical_H20mm, symbol Device:RotaryEncoder_Switch
Connections:
- net GND: now also volume_control1.C, volume_control1.S2
- net at R1.1: now also A1.17 (GPIO13); no longer A1.22 (GPIO17)
- net at D1.1: now also A1.19 (GPIO14); no longer A1.16 (GPIO12)
- net at Q1.1: now also A1.2 (GPIO1); no longer A1.20 (GPIO15)
- net at E1.1: now also A1.12 (GPIO9); no longer A1.17 (GPIO13)
- net at W1.1: now also A1.7 (GPIO5); no longer A1.19 (GPIO14)
- net at A1.21 (GPIO16): now also volume_control1.B; no longer F1.1
- net at A1.24 (GPIO18): now also volume_control1.A
- net at A1.26 (GPIO20): now also volume_control1.S1
- new net: A1.20 (GPIO15), F1.1
- no-connect marks 21 -> 13

Commit message: Complete Back Copper Routing
Connections:
- net at volume_control1.A: now also A1.25 (GPIO19); no longer A1.24 (GPIO18)
- net at volume_control1.B: now also A1.22 (GPIO17); no longer A1.21 (GPIO16)
- net at R1.1: now also A1.20 (GPIO15); no longer A1.17 (GPIO13)
- net at D1.1: now also A1.17 (GPIO13); no longer A1.19 (GPIO14)
- net at F1.1: now also A1.19 (GPIO14); no longer A1.20 (GPIO15)
- no-connect marks 13 -> 20
Changed lines of the file:
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@@
+	)
+	(junction
+		(at 80.01 80.01)
+		(diameter 0)
+		(color 0 0 0 0)
 	)
 	(junction
@@
 	)
 	(no_connect
+		(at 80.01 57.15)
+	)
+	(no_connect
 		(at 80.01 46.99)
 	)
@@
 	)
 	(no_connect
+		(at 80.01 72.39)
+	)
+	(no_connect
+		(at 80.01 62.23)
+	)
+	(no_connect
+		(at 80.01 74.93)
+	)
+	(no_connect
 		(at 125.73 77.47)
 	)
@@
 	)
 	(no_connect
+		(at 125.73 49.53)
+	)
+	(no_connect
 		(at 125.73 80.01)
 	)
@@
 	)
 	(no_connect
+		(at 125.73 54.61)
+	)
+	(no_connect
+		(at 80.01 77.47)
+	)
+	(no_connect
 		(at 125.73 62.23)
 	)
@@
 	(wire
 		(pts
-			(xy 80.01 137.16) (xy 80.01 85.09)
+			(xy 77.47 139.7) (xy 220.98 139.7)
+		)
+		(stroke
+			(width 0)
+			(type default)
+		)
+	)
+	(wire
+		(pts
+			(xy 76.2 137.16) (xy 203.2 137.16)
 		)
 		(stroke
@@
 	(wire
 		(pts
+			(xy 203.2 137.16) (xy 203.2 134.62)
+		)
+		(stroke
+			(width 0)
+			(type default)
+		)
+	)
+	(wire
+		(pts
 			(xy 158.75 129.54) (xy 71.12 129.54)
 		)
@@
 	(wire
 		(pts
-			(xy 135.89 49.53) (xy 125.73 49.53)
+			(xy 80.01 134.62) (xy 80.01 85.09)
 		)
 		(stroke
@@
 	(wire
 		(pts
-			(xy 140.97 33.02) (xy 140.97 54.61)
+			(xy 125.73 57.15) (xy 157.48 57.15)
+		)
+		(stroke
+			(width 0)
+			(type default)
+		)
+	)
+	(wire
+		(pts
+			(xy 80.01 80.01) (xy 81.28 80.01)
 		)
 		(stroke
@@
 	(wire
 		(pts
+			(xy 184.15 35.56) (xy 161.29 35.56)
+		)
+		(stroke
+			(width 0)
+			(type default)
+		)
+	)
+	(wire
+		(pts
+			(xy 203.2 105.41) (xy 186.69 105.41)
+		)
+		(stroke
+			(width 0)
+			(type default)
+		)
+	)
+	(wire
+		(pts
+			(xy 158.75 119.38) (xy 158.75 129.54)
+		)
+		(stroke
+			(width 0)
+			(type default)
+		)
+	)
+	(wire
+		(pts
+			(xy 204.47 105.41) (xy 203.2 105.41)
+		)
+		(stroke
+			(width 0)
+			(type default)
+		)
+	)
+	(wire
+		(pts
+			(xy 73.66 69.85) (xy 80.01 69.85)
+		)
+		(stroke
+			(width 0)
+			(type default)
+		)
+	)
+	(wire
+		(pts
+			(xy 76.2 80.01) (xy 76.2 137.16)
+		)
+		(stroke
+			(width 0)
+			(type default)
+		)
+	)
+	(wire
+		(pts
+			(xy 231.14 134.62) (xy 231.14 105.41)
+		)
+		(stroke
+			(width 0)
+			(type default)
+		)
+	)
+	(wire
+		(pts
+			(xy 176.53 119.38) (xy 176.53 127)
+		)
+		(stroke
+			(width 0)
+			(type default)
+		)
+	)
+	(wire
+		(pts
+			(xy 157.48 33.02) (xy 184.15 33.02)
+		)
+		(stroke
+			(width 0)
+			(type default)
+		)
+	)
+	(wire
+		(pts
+			(xy 161.29 105.41) (xy 168.91 105.41)
+		)
+		(stroke
+			(width 0)
+			(type default)
+		)
+	)
+	(wire
+		(pts
+			(xy 149.86 105.41) (xy 127 105.41)
+		)
+		(stroke
+			(width 0)
+			(type default)
+		)
+	)
+	(wire
+		(pts
+			(xy 184.15 38.1) (xy 184.15 52.07)
+		)
+		(stroke
+			(width 0)
+			(type default)
+		)
+	)
+	(wire
+		(pts
+			(xy 125.73 52.07) (xy 184.15 52.07)
+		)
+		(stroke
+			(width 0)
+			(type default)
+		)
+	)
+	(wire
+		(pts
+			(xy 176.53 127) (xy 73.66 127)
+		)
+		(stroke
+			(width 0)
+			(type default)
+		)
+	)
+	(wire
+		(pts
+			(xy 157.48 57.15) (xy 157.48 33.02)
+		)
+		(stroke
+			(width 0)
+			(type default)
+		)
+	)
+	(wire
+		(pts
+			(xy 213.36 105.41) (xy 204.47 105.41)
+		)
+		(stroke
+			(width 0)
+			(type default)
+		)
+	)
+	(wire
+		(pts
+			(xy 127 105.41) (xy 102.87 105.41)
+		)
+		(stroke
+			(width 0)
+			(type default)
+		)
+	)
+	(wire
+		(pts
 			(xy 76.2 80.01) (xy 80.01 80.01)
 		)
@@
 	(wire
 		(pts
-			(xy 184.15 35.56) (xy 161.29 35.56)
-		)
-		(stroke
-			(width 0)
-			(type default)
-		)
-	)
-	(wire
-		(pts
-			(xy 203.2 105.41) (xy 186.69 105.41)
-		)
-		(stroke
-			(width 0)
-			(type default)
-		)
-	)
-	(wire
-		(pts
-			(xy 135.89 38.1) (xy 135.89 49.53)
-		)
-		(stroke
-			(width 0)
-			(type default)
-		)
-	)
-	(wire
-		(pts
-			(xy 158.75 119.38) (xy 158.75 129.54)
-		)
-		(stroke
-			(width 0)
-			(type default)
-		)
-	)
-	(wire
-		(pts
-			(xy 204.47 105.41) (xy 203.2 105.41)
-		)
-		(stroke
-			(width 0)
-			(type default)
-		)
-	)
-	(wire
-		(pts
-			(xy 73.66 69.85) (xy 80.01 69.85)
-		)
-		(stroke
-			(width 0)
-			(type default)
-		)
-	)
-	(wire
-		(pts
-			(xy 194.31 133.35) (xy 76.2 133.35)
-		)
-		(stroke
-			(width 0)
-			(type default)
-		)
-	)
-	(wire
-		(pts
-			(xy 231.14 134.62) (xy 231.14 105.41)
-		)
-		(stroke
-			(width 0)
-			(type default)
-		)
-	)
-	(wire
-		(pts
-			(xy 194.31 119.38) (xy 194.31 133.35)
-		)
-		(stroke
-			(width 0)
-			(type default)
-		)
-	)
-	(wire
-		(pts
-			(xy 176.53 119.38) (xy 176.53 127)
-		)
-		(stroke
-			(width 0)
-			(type default)
-		)
-	)
-	(wire
-		(pts
-			(xy 184.15 33.02) (xy 140.97 33.02)
-		)
-		(stroke
-			(width 0)
-			(type default)
-		)
-	)
-	(wire
-		(pts
-			(xy 76.2 133.35) (xy 76.2 80.01)
-		)
-		(stroke
-			(width 0)
-			(type default)
-		)
-	)
-	(wire
-		(pts
-			(xy 161.29 105.41) (xy 168.91 105.41)
-		)
-		(stroke
-			(width 0)
-			(type default)
-		)
-	)
-	(wire
-		(pts
-			(xy 149.86 105.41) (xy 127 105.41)
-		)
-		(stroke
-			(width 0)
-			(type default)
-		)
-	)
-	(wire
-		(pts
-			(xy 184.15 38.1) (xy 135.89 38.1)
-		)
-		(stroke
-			(width 0)
-			(type default)
-		)
-	)
-	(wire
-		(pts
-			(xy 140.97 54.61) (xy 125.73 54.61)
-		)
-		(stroke
-			(width 0)
-			(type default)
-		)
-	)
-	(wire
-		(pts
-			(xy 176.53 127) (xy 73.66 127)
-		)
-		(stroke
-			(width 0)
-			(type default)
-		)
-	)
-	(wire
-		(pts
-			(xy 213.36 105.41) (xy 204.47 105.41)
-		)
-		(stroke
-			(width 0)
-			(type default)
-		)
-	)
-	(wire
-		(pts
-			(xy 127 105.41) (xy 102.87 105.41)
+			(xy 194.31 119.38) (xy 194.31 134.62)
 		)
 		(stroke
@@
 	(wire
 		(pts
-			(xy 220.98 137.16) (xy 80.01 137.16)
+			(xy 77.47 82.55) (xy 77.47 139.7)
 		)
 		(stroke
@@
 	(wire
 		(pts
-			(xy 220.98 134.62) (xy 220.98 137.16)
-		)
-		(stroke
-			(width 0)
-			(type default)
-		)
-	)
-	(wire
-		(pts
-			(xy 78.74 82.55) (xy 80.01 82.55)
+			(xy 220.98 134.62) (xy 220.98 139.7)
 		)
 		(stroke
@@
 	(wire
 		(pts
-			(xy 203.2 134.62) (xy 78.74 134.62)
+			(xy 80.01 82.55) (xy 77.47 82.55)
 		)
 		(stroke
@@
 	(wire
 		(pts
-			(xy 78.74 134.62) (xy 78.74 82.55)
-		)
-		(stroke
+			(xy 194.31 134.62) (xy 80.01 134.62)
+		)
+		(stroke
